Commit message: cleaned up granny model

File: catkin_ws/src/pnu_tb3open_launch/urdf/turtlebot_armed_granny.urdf.xacro (robot description, xacro)
@@ -38,5 +38,5 @@
     <parent link="base_link"/>
     <child link="wheel_front_left_link"/>
-    <origin xyz="0.129 0.1125 0.05" rpy="-1.57 0 0"/>
+    <origin xyz="0.1 0.1125 0.05" rpy="-1.57 0 0"/>
     <axis xyz="0 0 1"/>
   </joint>
@@ -66,5 +66,5 @@
     <parent link="base_link"/>
     <child link="wheel_front_right_link"/>
-    <origin xyz="0.129 -0.1125 0.05" rpy="-1.57 0 0"/>
+    <origin xyz="0.1 -0.1125 0.05" rpy="-1.57 0 0"/>
     <axis xyz="0 0 1"/>
   </joint>
@@ -94,5 +94,5 @@
     <parent link="base_link"/>
     <child link="wheel_back_left_link"/>
-    <origin xyz="-0.129 0.1125 0.05" rpy="-1.57 0 0"/>
+    <origin xyz="-0.1 0.1125 0.05" rpy="-1.57 0 0"/>
     <axis xyz="0 0 1"/>
   </joint>
@@ -122,5 +122,5 @@
     <parent link="base_link"/>
     <child link="wheel_back_right_link"/>
-    <origin xyz="-0.129 -0.1125 0.05" rpy="1.57 0 0"/>
+    <origin xyz="-0.1 -0.1125 0.05" rpy="1.57 0 0"/>
     <axis xyz="0 0 1"/>
   </joint>

Commit message: 2021 update

File: catkin_ws/src/pnu_tb3open_launch/urdf/turtlebot_armed_granny.urdf.xacro (robot description, xacro)
@@ -9,11 +9,9 @@
   </joint>
   <link name="base_link">
-    <!-- <visual>
-      <origin xyz="0 0 0.0" rpy="0 0 0"/>
-      <geometry>
-        <mesh filename="package://pnu_tb3_launch/meshes/bases/burger_base.stl" scale="0.001 0.001 0.001"/>
-      </geometry>
-      <material name="light_black"/>
-    </visual> -->
+    <origin xyz="0 0 0.0" rpy="0 0 0"/>
+    <geometry>
+      <mesh filename="package://pnu_tb3_launch/meshes/bases/burger_base.stl" scale="0.001 0.001 0.001"/>
+    </geometry>
+    <material name="light_black"/>
     <collision>
       <origin xyz="0.032 0 0.070" rpy="0 0 0"/>
@@ -33,10 +31,10 @@
     <parent link="base_footprint"/>
     <child link="arm_base_link"/>
-    <origin xyz="-0.06 0.0 0.15" rpy="0 0 0"/>
+    <origin xyz="0.108 0.0 0.15" rpy="0 0 0"/>
   </joint>
   <joint name="wheel1" type="continuous">
     <parent link="base_link"/>
     <child link="wheel_front_left_link"/>
-    <origin xyz="0.1 0.1125 0.05" rpy="-1.57 0 0"/>
+    <origin xyz="0.0925 0.1125 0.05" rpy="-1.57 0 0"/>
     <axis xyz="0 0 1"/>
   </joint>
@@ -66,5 +64,5 @@
     <parent link="base_link"/>
     <child link="wheel_front_right_link"/>
-    <origin xyz="0.1 -0.1125 0.05" rpy="-1.57 0 0"/>
+    <origin xyz="0.0925 -0.1125 0.05" rpy="-1.57 0 0"/>
     <axis xyz="0 0 1"/>
   </joint>
@@ -94,5 +92,5 @@
     <parent link="base_link"/>
     <child link="wheel_back_left_link"/>
-    <origin xyz="-0.1 0.1125 0.05" rpy="-1.57 0 0"/>
+    <origin xyz="-0.0925 0.1125 0.05" rpy="-1.57 0 0"/>
     <axis xyz="0 0 1"/>
   </joint>
@@ -122,5 +120,5 @@
     <parent link="base_link"/>
     <child link="wheel_back_right_link"/>
-    <origin xyz="-0.1 -0.1125 0.05" rpy="1.57 0 0"/>
+    <origin xyz="-0.0925 -0.1125 0.05" rpy="1.57 0 0"/>
     <axis xyz="0 0 1"/>
   </joint>
@@ -168,5 +166,6 @@
     <parent link="base_link"/>
     <child link="base_scan"/>
-    <origin xyz="0.073 0 0.155" rpy="0 0 0"/>
+    <!-- <origin xyz="0.073 0 0.155" rpy="0 0 0"/> -->
+    <origin xyz="-0.095 0 0.155" rpy="0 0 0"/>
   </joint>
   <link name="base_scan">
