Commit message: update to noetic

File: catkin_ws/src/pnu_tb3open_launch/urdf/turtlebot3_burger.urdf.xacro (robot description, xacro)
@@ -1,5 +1,5 @@
 <?xml version="1.0" ?>
 <robot name="turtlebot3_burger" xmlns:xacro="http://ros.org/wiki/xacro">
-  <xacro:include filename="$(find pnu_tb3_launch)/urdf/common_properties.xacro"/>
+  <xacro:include filename="$(find pnu_tb3open_launch)/urdf/common_properties.xacro"/>
   <link name="base_footprint"/>
   <joint name="base_joint" type="fixed">
@@ -12,5 +12,5 @@
       <origin xyz="-0.032 0 0.0" rpy="0 0 0"/>
       <geometry>
-        <mesh filename="package://pnu_tb3_launch/meshes/bases/burger_base.stl" scale="0.001 0.001 0.001"/>
+        <mesh filename="package://pnu_tb3open_launch/meshes/bases/burger_base.stl" scale="0.001 0.001 0.001"/>
       </geometry>
       <material name="light_black"/>
@@ -52,5 +52,5 @@
       <origin xyz="0 0 0" rpy="1.57 0 0"/>
       <geometry>
-        <mesh filename="package://pnu_tb3_launch/meshes/wheels/left_tire.stl" scale="0.001 0.001 0.001"/>
+        <mesh filename="package://pnu_tb3open_launch/meshes/wheels/left_tire.stl" scale="0.001 0.001 0.001"/>
       </geometry>
       <material name="dark"/>
@@ -80,5 +80,5 @@
       <origin xyz="0 0 0" rpy="1.57 0 0"/>
       <geometry>
-        <mesh filename="package://pnu_tb3_launch/meshes/wheels/right_tire.stl" scale="0.001 0.001 0.001"/>
+        <mesh filename="package://pnu_tb3open_launch/meshes/wheels/right_tire.stl" scale="0.001 0.001 0.001"/>
       </geometry>
       <material name="dark"/>
@@ -133,5 +133,5 @@
       <origin xyz="0 0 0.0" rpy="0 0 0"/>
       <geometry>
-        <mesh filename="package://pnu_tb3_launch/meshes/sensors/lds.stl" scale="0.001 0.001 0.001"/>
+        <mesh filename="package://pnu_tb3open_launch/meshes/sensors/lds.stl" scale="0.001 0.001 0.001"/>
       </geometry>
       <material name="dark"/>

File: catkin_ws/src/pnu_tb3open_launch/urdf/turtlebot_armed_granny.urdf.xacro (robot description, xacro)
@@ -1,5 +1,5 @@
 <?xml version="1.0" ?>
 <robot name="turtlebot_armed_granny" xmlns:xacro="http://ros.org/wiki/xacro">
-  <xacro:include filename="$(find pnu_tb3_launch)/urdf/common_properties.xacro"/>
+  <xacro:include filename="$(find pnu_tb3open_launch)/urdf/common_properties.xacro"/>
   <link name="base_footprint"/>
   <joint name="base_joint" type="fixed">
@@ -11,5 +11,5 @@
     <origin xyz="0 0 0.0" rpy="0 0 0"/>
     <geometry>
-      <mesh filename="package://pnu_tb3_launch/meshes/bases/burger_base.stl" scale="0.001 0.001 0.001"/>
+      <mesh filename="package://pnu_tb3open_launch/meshes/bases/burger_base.stl" scale="0.001 0.001 0.001"/>
     </geometry>
     <material name="light_black"/>
@@ -43,5 +43,5 @@
       <origin xyz="0 0 0" rpy="1.57 0 0"/>
       <geometry>
-        <mesh filename="package://pnu_tb3_launch/meshes/wheels/left_tire.stl" scale="0.001 0.001 0.001"/>
+        <mesh filename="package://pnu_tb3open_launch/meshes/wheels/left_tire.stl" scale="0.001 0.001 0.001"/>
       </geometry>
       <material name="dark"/>
@@ -71,5 +71,5 @@
       <origin xyz="0 0 0" rpy="1.57 0 0"/>
       <geometry>
-        <mesh filename="package://pnu_tb3_launch/meshes/wheels/right_tire.stl" scale="0.001 0.001 0.001"/>
+        <mesh filename="package://pnu_tb3open_launch/meshes/wheels/right_tire.stl" scale="0.001 0.001 0.001"/>
       </geometry>
       <material name="dark"/>
@@ -99,5 +99,5 @@
       <origin xyz="0 0 0" rpy="1.57 0 0"/>
       <geometry>
-        <mesh filename="package://pnu_tb3_launch/meshes/wheels/left_tire.stl" scale="0.001 0.001 0.001"/>
+        <mesh filename="package://pnu_tb3open_launch/meshes/wheels/left_tire.stl" scale="0.001 0.001 0.001"/>
       </geometry>
       <material name="dark"/>
@@ -127,5 +127,5 @@
       <origin xyz="0 0 0" rpy="1.57 0 0"/>
       <geometry>
-        <mesh filename="package://pnu_tb3_launch/meshes/wheels/right_tire.stl" scale="0.001 0.001 0.001"/>
+        <mesh filename="package://pnu_tb3open_launch/meshes/wheels/right_tire.stl" scale="0.001 0.001 0.001"/>
       </geometry>
       <material name="dark"/>
@@ -173,5 +173,5 @@
       <origin xyz="0 0 0.0" rpy="0 0 0"/>
       <geometry>
-        <mesh filename="package://pnu_tb3_launch/meshes/sensors/lds.stl" scale="0.001 0.001 0.001"/>
+        <mesh filename="package://pnu_tb3open_launch/meshes/sensors/lds.stl" scale="0.001 0.001 0.001"/>
       </geometry>
       <material name="dark"/>
@@ -196,12 +196,12 @@
       <origin xyz="0 0 0" rpy="0 0 0"/>
       <geometry>
-        <mesh filename="package://pnu_tb3_launch/meshes/manipulator/chain_link1.stl" scale="0.001 0.001 0.001"/>
-      </geometry>
-      <material name="grey"/>
-    </visual>
-    <collision>
-      <origin xyz="0 0 0" rpy="0 0 0"/>
-      <geometry>
-        <mesh filename="package://pnu_tb3_launch/meshes/manipulator/chain_link1.stl" scale="0.001 0.001 0.001"/>
+        <mesh filename="package://pnu_tb3open_launch/meshes/manipulator/chain_link1.stl" scale="0.001 0.001 0.001"/>
+      </geometry>
+      <material name="grey"/>
+    </visual>
+    <collision>
+      <origin xyz="0 0 0" rpy="0 0 0"/>
+      <geometry>
+        <mesh filename="package://pnu_tb3open_launch/meshes/manipulator/chain_link1.stl" scale="0.001 0.001 0.001"/>
       </geometry>
     </collision>
@@ -227,5 +227,5 @@
       <origin xyz="0 0 0.019" rpy="0 0 0"/>
       <geometry>
-        <mesh filename="package://pnu_tb3_launch/meshes/manipulator/chain_link2.stl" scale="0.001 0.001 0.001"/>
+        <mesh filename="package://pnu_tb3open_launch/meshes/manipulator/chain_link2.stl" scale="0.001 0.001 0.001"/>
       </geometry>
       <material name="grey"/>
@@ -234,5 +234,5 @@
       <origin xyz="0 0 0.019" rpy="0 0 0"/>
       <geometry>
-        <mesh filename="package://pnu_tb3_launch/meshes/manipulator/chain_link2.stl" scale="0.001 0.001 0.001"/>
+        <mesh filename="package://pnu_tb3open_launch/meshes/manipulator/chain_link2.stl" scale="0.001 0.001 0.001"/>
       </geometry>
     </collision>
@@ -258,12 +258,12 @@
       <origin xyz="0 0 0" rpy="0 0 0"/>
       <geometry>
-        <mesh filename="package://pnu_tb3_launch/meshes/manipulator/chain_link3.stl" scale="0.001 0.001 0.001"/>
-      </geometry>
-      <material name="grey"/>
-    </visual>
-    <collision>
-      <origin xyz="0 0 0" rpy="0 0 0"/>
-      <geometry>
-        <mesh filename="package://pnu_tb3_launch/meshes/manipulator/chain_link3.stl" scale="0.001 0.001 0.001"/>
+        <mesh filename="package://pnu_tb3open_launch/meshes/manipulator/chain_link3.stl" scale="0.001 0.001 0.001"/>
+      </geometry>
+      <material name="grey"/>
+    </visual>
+    <collision>
+      <origin xyz="0 0 0" rpy="0 0 0"/>
+      <geometry>
+        <mesh filename="package://pnu_tb3open_launch/meshes/manipulator/chain_link3.stl" scale="0.001 0.001 0.001"/>
       </geometry>
     </collision>
@@ -289,12 +289,12 @@
       <origin xyz="0 0 0" rpy="0 0 0"/>
       <geometry>
-        <mesh filename="package://pnu_tb3_launch/meshes/manipulator/chain_link4.stl" scale="0.001 0.001 0.001"/>
-      </geometry>
-      <material name="grey"/>
-    </visual>
-    <collision>
-      <origin xyz="0 0 0" rpy="0 0 0"/>
-      <geometry>
-        <mesh filename="package://pnu_tb3_launch/meshes/manipulator/chain_link4.stl" scale="0.001 0.001 0.001"/>
+        <mesh filename="package://pnu_tb3open_launch/meshes/manipulator/chain_link4.stl" scale="0.001 0.001 0.001"/>
+      </geometry>
+      <material name="grey"/>
+    </visual>
+    <collision>
+      <origin xyz="0 0 0" rpy="0 0 0"/>
+      <geometry>
+        <mesh filename="package://pnu_tb3open_launch/meshes/manipulator/chain_link4.stl" scale="0.001 0.001 0.001"/>
       </geometry>
     </collision>
@@ -320,12 +320,12 @@
       <origin xyz="0 0 0" rpy="0 0 0"/>
       <geometry>
-        <mesh filename="package://pnu_tb3_launch/meshes/manipulator/chain_link5.stl" scale="0.001 0.001 0.001"/>
-      </geometry>
-      <material name="grey"/>
-    </visual>
-    <collision>
-      <origin xyz="0 0 0" rpy="0 0 0"/>
-      <geometry>
-        <mesh filename="package://pnu_tb3_launch/meshes/manipulator/chain_link5.stl" scale="0.001 0.001 0.001"/>
+        <mesh filename="package://pnu_tb3open_launch/meshes/manipulator/chain_link5.stl" scale="0.001 0.001 0.001"/>
+      </geometry>
+      <material name="grey"/>
+    </visual>
+    <collision>
+      <origin xyz="0 0 0" rpy="0 0 0"/>
+      <geometry>
+        <mesh filename="package://pnu_tb3open_launch/meshes/manipulator/chain_link5.stl" scale="0.001 0.001 0.001"/>
       </geometry>
     </collision>
@@ -352,5 +352,5 @@
       <origin xyz="0.0 0.0 0" rpy="0 0 0"/>
       <geometry>
-        <mesh filename="package://pnu_tb3_launch/meshes/manipulator/chain_link_grip_l.stl" scale="0.001 0.001 0.001"/>
+        <mesh filename="package://pnu_tb3open_launch/meshes/manipulator/chain_link_grip_l.stl" scale="0.001 0.001 0.001"/>
       </geometry>
       <material name="grey"/>
@@ -359,5 +359,5 @@
       <origin xyz="0.0 0.0 0" rpy="0 0 0"/>
       <geometry>
-        <mesh filename="package://pnu_tb3_launch/meshes/manipulator/chain_link_grip_l.stl" scale="0.001 0.001 0.001"/>
+        <mesh filename="package://pnu_tb3open_launch/meshes/manipulator/chain_link_grip_l.stl" scale="0.001 0.001 0.001"/>
       </geometry>
     </collision>
@@ -385,5 +385,5 @@
       <origin xyz="0.0 -0.0 0" rpy="0 0 0"/>
       <geometry>
-        <mesh filename="package://pnu_tb3_launch/meshes/manipulator/chain_link_grip_r.stl" scale="0.001 0.001 0.001"/>
+        <mesh filename="package://pnu_tb3open_launch/meshes/manipulator/chain_link_grip_r.stl" scale="0.001 0.001 0.001"/>
       </geometry>
       <material name="grey"/>
@@ -392,5 +392,5 @@
       <origin xyz="0.0 -0.0 0" rpy="0 0 0"/>
       <geometry>
-        <mesh filename="package://pnu_tb3_launch/meshes/manipulator/chain_link_grip_r.stl" scale="0.001 0.001 0.001"/>
+        <mesh filename="package://pnu_tb3open_launch/meshes/manipulator/chain_link_grip_r.stl" scale="0.001 0.001 0.001"/>
       </geometry>
     </collision>
